Commit message: mover

File: codigo/ros2_ws/src/mi_ackermann_description/urdf/mobile_base.xacro (robot description, xacro)
@@ -5,14 +5,20 @@
   <xacro:property name="PI" value="3.1415926535897931"/>
   <xacro:property name="base_mass" value="4.0" /> <!-- arbitrary value for base mass -->
-  <xacro:property name="base_width" value="0.12" />
-  <xacro:property name="base_length" value="0.15" />
+  <xacro:property name="base_width" value="0.260" />
+  <xacro:property name="base_length" value="0.525" />
   <xacro:property name="base_height" value="0.060" />
-  <xacro:property name="wheelbase" value="0.12" />
+  <xacro:property name="wheelbase" value="0.325" />
   <xacro:property name="wheel_mass" value="0.34055" /> <!-- arbitrary value for wheel mass -->
-  <xacro:property name="wheel_len" value="0.02" />
-  <xacro:property name="wheel_radius" value="0.02" />
+  <xacro:property name="wheel_len" value="0.045" />
+  <xacro:property name="wheel_radius" value="0.05" />
   <!-- <xacro:property name="wheeltrack" value="" -->
   <!-- Base Link -->
   <link name="${prefix}base_link" />
+  <joint name="${prefix}base_footprint_joint" type="fixed">
+      <parent link="${prefix}base_link"/>
+      <child link="${prefix}base_footprint"/>
+      <origin xyz="0 0 0" rpy="0 0 0"/>
+  </joint>
+  <link name="${prefix}base_footprint" />
   <!-- Chassis -->
   <link name="${prefix}chassis_link">
@@ -56,4 +62,9 @@
         <material name="invisible"/>
       </visual>
+      <inertial>
+    <origin xyz="0 0 0" rpy="0 0 0"/>
+    <mass value="0.001"/>
+    <inertia ixx="1e-6" ixy="0.0" ixz="0.0" iyy="1e-6" iyz="0.0" izz="1e-6"/>
+  </inertial>
     </link>
     <joint name="${prefix}virtual_rear_wheel_joint" type="continuous">
@@ -141,4 +152,9 @@
         <material name="invisible"/>
       </visual>
+      <inertial>
+    <origin xyz="0 0 0" rpy="0 0 0"/>
+    <mass value="0.001"/>
+    <inertia ixx="1e-6" ixy="0.0" ixz="0.0" iyy="1e-6" iyz="0.0" izz="1e-6"/>
+  </inertial>
     </link>
     <joint name="${prefix}virtual_front_wheel_joint" type="revolute">
@@ -216,22 +232,4 @@
       <mimic joint="${prefix}virtual_front_wheel_joint" multiplier="1.0" offset="0.0"/>
     </joint>
-  <!-- ====================== -->
-  <!-- LiDAR -->
-  <!-- ====================== -->
-  <link name="${prefix}laser">
-    <visual>
-      <geometry>
-        <cylinder radius="0.03" length="0.04"/>
-      </geometry>
-      <material name="black"/>
-    </visual>
-  </link>
-  <joint name="${prefix}laser_joint" type="fixed">
-    <parent link="${prefix}base_link"/>
-    <child link="${prefix}laser"/>
-    <!-- Ajustar según la posición real -->
-    <origin xyz="0.25 0.06 0.17"
-            rpy="0 0 0"/>
-  </joint>
   </xacro:macro>
 </robot>

File: codigo/ros2_ws/src/mi_ackermann_description/urdf/mobile_baseg.ros2_control.xacro (robot description, xacro)
@@ -5,31 +5,35 @@
     <ros2_control name="CarLikeSystem" type="system">
       <hardware>
-        <!-- =================== MOCK =================== -->
+        <!-- MOCK -->
         <xacro:if value="${hardware_type == 'mock'}">
           <plugin>mock_components/GenericSystem</plugin>
         </xacro:if>
-        <!-- =================== GAZEBO =================== -->
+        <!-- GAZEBO -->
         <xacro:if value="${hardware_type == 'gazebo'}">
           <plugin>gz_ros2_control/GazeboSimSystem</plugin>
         </xacro:if>
-        <!-- =================== ROBOT REAL =================== -->
+        <!-- HARDWARE REAL -->
         <xacro:if value="${hardware_type == 'real'}">
           <plugin>mi_ackermann_hardware/AckermannHardware</plugin>
-          <param name="ip">192.168.0.110</param>
-          <param name="port">1300</param>
+          <param name="ip">192.168.0.103</param>
+          <param name="port">12348</param>
           <param name="traction_type">large</param>
         </xacro:if>
       </hardware>
-      <!-- Dirección -->
-      <joint name="${prefix}virtual_front_wheel_joint">
+      <!-- ================================= -->
+      <!-- Steering wheel                    -->
+      <!-- ================================= -->
+      <joint name="${prefix}front_wheel_joint">
         <command_interface name="position"/>
         <state_interface name="position"/>
         <state_interface name="velocity"/>
       </joint>
-      <!-- Tracción -->
-      <joint name="${prefix}virtual_rear_wheel_joint">
+      <!-- ================================= -->
+      <!-- Traction wheel                    -->
+      <!-- ================================= -->
+      <joint name="${prefix}rear_wheel_joint">
         <command_interface name="velocity"/>
+        <state_interface name="position"/>
         <state_interface name="velocity"/>
-        <state_interface name="position"/>
       </joint>
     </ros2_control>

File: codigo/ros2_ws/src/mi_ackermann_description/urdf/my_robotg.urdf.xacro (robot description, xacro)
@@ -2,6 +2,6 @@
 <robot xmlns:xacro="http://www.ros.org/wiki/xacro" name="my_robot">
   <xacro:include filename="common_propperties.xacro"/>
-  <xacro:include filename="mobile_base.xacro"/>
-  <xacro:include filename="mobile_base.ros2_control.xacro"/>
+  <xacro:include filename="mobile_baseg.xacro"/>
+  <xacro:include filename="mobile_baseg.ros2_control.xacro"/>
   <xacro:include filename="mobile_base.gazebo.xacro"/>
   <!-- instancia el robot -->
@@ -10,5 +10,5 @@
   <xacro:carlikebot_ros2_control
     prefix=""
-    hardware_type="real"/>
+    hardware_type="gazebo"/>
   <xacro:carlikebot_gazebo prefix=""/>
 </robot>

File: codigo/ros2_ws/src/mi_ackermann_description_viz/urdf/mobile_base.xacro (robot description, xacro)
@@ -5,11 +5,11 @@
   <xacro:property name="PI" value="3.1415926535897931"/>
   <xacro:property name="base_mass" value="4.0" />
-  <xacro:property name="base_width" value="0.260" />
-  <xacro:property name="base_length" value="0.525" />
+  <xacro:property name="base_width" value="0.12" />
+  <xacro:property name="base_length" value="0.15" />
   <xacro:property name="base_height" value="0.060" />
-  <xacro:property name="wheelbase" value="0.325" />
+  <xacro:property name="wheelbase" value="0.12" />
   <xacro:property name="wheel_mass" value="0.34055" />
-  <xacro:property name="wheel_len" value="0.045" />
-  <xacro:property name="wheel_radius" value="0.05" />
+  <xacro:property name="wheel_len" value="0.02" />
+  <xacro:property name="wheel_radius" value="0.02" />
   <!-- Base Link -->
   <link name="${prefix}base_link" />
