Commit message: SLAM

File: codigo/ros2_ws/src/mi_ackermann_description/urdf/mobile_base.ros2_control.xacro (robot description, xacro)
@@ -17,5 +17,5 @@
           <plugin>mi_ackermann_hardware/AckermannHardware</plugin>
           <param name="ip">192.168.0.110</param>
-          <param name="port">1300</param>
+          <param name="port">2100</param>
           <param name="traction_type">large</param>
         </xacro:if>

File: codigo/ros2_ws/src/mi_ackermann_description/urdf/mobile_base.xacro (robot description, xacro)
@@ -5,11 +5,11 @@
   <xacro:property name="PI" value="3.1415926535897931"/>
   <xacro:property name="base_mass" value="4.0" /> <!-- arbitrary value for base mass -->
-  <xacro:property name="base_width" value="0.260" />
-  <xacro:property name="base_length" value="0.525" />
-  <xacro:property name="base_height" value="0.060" />
-  <xacro:property name="wheelbase" value="0.325" />
+  <xacro:property name="base_width" value="0.20" />
+  <xacro:property name="base_length" value="0.35" />
+  <xacro:property name="base_height" value="0.24" />
+  <xacro:property name="wheelbase" value="0.15" />
   <xacro:property name="wheel_mass" value="0.34055" /> <!-- arbitrary value for wheel mass -->
   <xacro:property name="wheel_len" value="0.045" />
-  <xacro:property name="wheel_radius" value="0.05" />
+  <xacro:property name="wheel_radius" value="0.02" />
   <!-- <xacro:property name="wheeltrack" value="" -->
   <!-- Base Link -->
